Commit message: romi initial commit

File: my_robot_description/urdf/macros.urdf.xacro (robot description, xacro)
@@ -1,7 +1,4 @@
 <?xml version="1.0"?>
-<!--
-	definitions of some macros for easier description of the robot
--->
-<robot xmlns:xacro="http://www.ros.org/wiki/xacro">
+<robot name="my_robot_macros" xmlns:xacro="http://www.ros.org/wiki/xacro">
   <xacro:macro name="cylinder_inertia" params="m r h">
     <inertia
@@ -85,7 +82,4 @@
       <joint_properties damping="0.0" friction="0.0"/>
     </joint>
-<!--
-  http://gazebosim.org/tutorials/?tut=ros_control
--->
     <transmission name="${lr}_trans">
       <type>transmission_interface/SimpleTransmission</type>

File: my_robot_description/urdf/materials.urdf.xacro (robot description, xacro)
@@ -3,5 +3,5 @@
 	definition of the materials used
 -->
-<robot>
+<robot name="my_robot_materials" xmlns:xacro="http://ros.org/wiki/xacro">
 	<material name="black">
 	  <color rgba="0.0 0.0 0.0 1.0"/>

File: my_robot_description/urdf/my_robot.urdf.xacro (robot description, xacro)
@@ -1,24 +1,14 @@
 <?xml version="1.0"?>
-<!--
-	http://www.generationrobots.com/blog/en/2015/02/robotic-simulation-scenarios-with-gazebo-and-ros/#create your own robot model
-	#######################################################
-    To run:
-    $ roslaunch my_robot_gazebo my_robot_world.launch paused:=true
-    $ rosrun turtlebot_teleop turtlebot_teleop_key /turtlebot_teleop/cmd_vel:=/my_robot/cmd_vel
--->
 <robot name="my_robot" xmlns:xacro="http://www.ros.org/wiki/xacro">
-	<!-- Robot constants and properties -->
-	<xacro:include filename="$(find my_robot_description)/urdf/my_robot_properties.xacro" />
-	<!-- Import Rviz colors -->
-	<xacro:include filename="$(find my_robot_description)/urdf/materials.xacro" />
-	<!-- Gazebo aspects of the robot -->
-	<xacro:include filename="$(find my_robot_description)/urdf/my_robot.gazebo" />
-	<!-- Inertia matrices -->
-	<xacro:include filename="$(find my_robot_description)/urdf/macros.xacro" />
+	<xacro:include filename="$(find my_robot_description)/urdf/my_robot_properties.urdf.xacro" />
+	<!-- <xacro:include filename="$(find my_robot_description)/urdf/materials.urdf.xacro" /> -->
+	<xacro:include filename="$(find my_robot_description)/urdf/my_robot.gazebo.xacro"/>
+	<!-- <xacro:include filename="$(find my_robot_description)/urdf/macros.urdf.xacro" /> -->
 	<!-- Used for fixing robot to Gazebo 'chassis' -->
-	<link name="base_footprint" />
+	<link name="base_footprint"/>
 	<joint name="base_joint" type="fixed">
 		<parent link="base_footprint"/>
 		<child link="chassis"/>
+		<origin xyz="0.0 0.0 0.010" rpy="0 0 0"/>
 	</joint>
 	<link name='chassis'>
@@ -27,5 +17,5 @@
 					rpy="0 0 0"/>
 			<geometry>
-				<mesh filename="package://my_robot_description/meshes/chassis.dae" />
+				<mesh filename="package://my_robot_description/meshes/chassis.dae"/>
 			</geometry>
 		</collision>
@@ -34,5 +24,5 @@
 					rpy="0 0 0"/>
 			<geometry>
-				<mesh filename="package://my_robot_description/meshes/chassis.dae" />
+				<mesh filename="package://my_robot_description/meshes/chassis.dae"/>
 			</geometry>
 			<material name="red"/>
@@ -58,5 +48,5 @@
 					rpy="0 0 0"/>
 			<geometry>
-				<mesh filename="package://my_robot_description/meshes/caster_wheel.dae" />
+				<mesh filename="package://my_robot_description/meshes/caster_wheel.dae"/>
 	  		</geometry>
 		</collision>
@@ -65,7 +55,7 @@
 					rpy="0 0 0"/>
 			<geometry>
-				<mesh filename="package://my_robot_description/meshes/caster_wheel.dae" />
+				<mesh filename="package://my_robot_description/meshes/caster_wheel.dae"/>
 			</geometry>
-			<material name="grey" />
+			<material name="grey"/>
 		</visual>
 		<inertial>
@@ -81,4 +71,4 @@
 	<wheel lr="right" tY="1"/>
 	<!-- Sensor models -->
-	<xacro:include filename="$(find my_robot_description)/urdf/sensors.xacro" />
+	<!-- <xacro:include filename="$(find my_robot_description)/urdf/sensors.urdf.xacro"/> -->
 </robot>

File: my_robot_description/urdf/my_robot_properties.urdf.xacro (robot description, xacro)
@@ -1,4 +1,4 @@
 <?xml version="1.0"?>
-<robot xmlns:xacro="http://www.ros.org/wiki/xacro">
+<robot name="my_robot_properties" xmlns:xacro="http://www.ros.org/wiki/xacro">
 	<!-- Constants -->
 	<xacro:property name="PI" value="3.1415926535897931"/>

File: my_robot_description/urdf/sensors.urdf.xacro (robot description, xacro)
@@ -1,18 +1,7 @@
 <?xml version="1.0" ?>
-<!--
-  https://www.youtube.com/watch?v=HIK1KBw-Jn4
-  http://moorerobots.com/blog/post/3
-  https://github.com/richardw05/mybot_ws/tree/master/src
-  https://github.com/qboticslabs/Chefbot_ROS_pkg
-  https://answers.ros.org/question/249568/no-such-file-or-directory-gmappinglaunchxml-or-amcllaunchxml-under-turtlebot_navigationlaunchincludes/
-  http://wiki.ros.org/navigation/Tutorials
--->
-<robot xmlns:xacro="http://www.ros.org/wiki/xacro">
-  <!-- Robot constants and properties -->
-  <xacro:include filename="$(find my_robot_description)/urdf/my_robot_properties.xacro" />
-  <!-- Inertia matrices -->
+<robot name="my_robot_sensors" xmlns:xacro="http://www.ros.org/wiki/xacro">
+  <!-- <xacro:include filename="$(find my_robot_description)/urdf/my_robot_properties.xacro" />
   <xacro:include filename="$(find my_robot_description)/urdf/macros.xacro" />
-  <!-- Gazebo aspects of the robot -->
-  <xacro:include filename="$(find my_robot_description)/urdf/my_robot.gazebo" />
+  <xacro:include filename="$(find my_robot_description)/urdf/my_robot.gazebo" /> -->
   <link name="camera_link">
     <collision>
